Commit message: Add Hokuyo LiDAR, OctoMap, and Hector SLAM support

File: src/mushr_description/urdf/racecar.urdf (robot description, URDF)
Before this commit: robot mushr_tx2, 13 links, 12 joints
Links:
- added link laser_link; visual cylinder length=0.04 radius=0.03
Joints:
- added joint laser_joint: type fixed, parent base_link, child laser_link, origin xyz=0.15 0 0.15 rpy=0 0 0
